Commit message: Fix bugs

File: model/add.urdf (robot description, URDF)
Before this commit: robot spawn_objects, 1 links, 0 joints
Links:
- removed link worldbody
- added link Object_0; collision box size=0.005156 0.320000 0.335000; collision box size=0.005156 0.320000 0.335000
- added link box_top_layer_bottom; collision mesh filename=package://mujoco_sim/model/tmp/../../../mujoco_world/mujoco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
- added link box_top_layer_top; collision mesh filename=package://mujoco_sim/model/tmp/../../../mujoco_world/mujoco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
- added link odom
Joints:
- added joint Object_0_joint: type fixed, parent odom, child Object_0
- added joint box_top_layer_bottom_joint: type continuous, parent Object_0, child box_top_layer_bottom, origin xyz=0.17 0 0.166 rpy=0 0 0, axis 0 1 0
- added joint box_top_layer_top_joint: type continuous, parent Object_0, child box_top_layer_top, origin xyz=-0.17 0 0.168 rpy=0 0 0, axis 0 -1 0
